File: KiCAD_Files/Transmitter-Remote-Control/Transmitter-Remote-Control.kicad_pcb (KiCad board)
At the start: 2 copper layers, 100 x 100 mm, 30 parts, among them J1 PWR_IN, J2 MPU6050, J3 NOKIA 5110, J4 ICSP, SW1 PWR_SW, SW2 RESET, SW3 BUTTON, SW4 SW1, SW5 SW2, U1 LM1117-3.3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

Commit message: Update hardware.
Parts:
- U4: footprint Package_DIP:DIP-42_W15.24mm_LongPads -> Package_DIP:DIP-40_W15.24mm_LongPads
- moved C7 4.84 mm to (147.0, 148.3)
Routing:
- net RST: track 45.9 -> 62.2 mm, vias 2 -> 4
- net CE_Nokia: track 64.3 -> 75.9 mm
- net DC: track 138.9 -> 144.8 mm
- net PGC: track 54.0 -> 48.9 mm
- net PGD: track 37.9 -> 32.8 mm
- net ~CSN: track 109.8 -> 106.1 mm
- net CE: track 68.1 -> 65.0 mm
- net +5V: track 245.7 -> 248.5 mm
- net SDA: track 91.0 -> 93.1 mm
- net DIN: track 221.2 -> 222.7 mm
- net GND: track 286.0 -> 286.5 mm
